File: hardware/v0.2/bed-lift.kicad_sch (KiCad schematic)
At the start: 43 parts, among them J1 SM04B-SRSS-TB, J2 S2P-VH, J3 SM04B-SRSS-TB, J4 TC2030-NL, J5 PH1-06-UA, J6 S3B-XH-A, J7 S6B-XH-A, U1 LP2985-33DBVR, U2 ISO1640, U3 STM32C031K6T6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

Commit message: Finalize for production
Parts:
- C1, C2: LCSC C15849 -> C14663
- D1: Alternative SMF16A-E3-08 -> (none); FT Rotation Offset (none) -> 180; LCSC C207257 -> C74561
- J2: FT Rotation Offset (none) -> 180; LCSC (none) -> C160355
- J5: now not fitted; now left out of the parts list
- J6: FT Rotation Offset (none) -> 180; LCSC (none) -> C157928
- J7: FT Rotation Offset (none) -> 180; LCSC (none) -> C157919
- U2, U4: FT Rotation Offset (none) -> 90
Connections:
- net +3.3V: now also U2.1 (VCC1); no longer U2.8 (VCC2)
- net BUS_3V3: now also U2.8 (VCC2); no longer U2.1 (VCC1)
- net BUS_GND: now also U2.5 (GND2); no longer U2.4 (GND1)
- net BUS_SCL: now also U2.6 (SCL2); no longer U2.3 (SCL1)
- net BUS_SDA: now also U2.7 (SDA2); no longer U2.2 (SDA1)
- net GND: now also U2.4 (GND1); no longer U2.5 (GND2)
- net I2C1_SCL: now also U2.3 (SCL1); no longer U2.6 (SCL2)
- net I2C1_SDA: now also U2.2 (SDA1); no longer U2.7 (SDA2)
Other:
- note added: "ISO1640 provides bidirectional isolation, hot swap, and ESD protection - Side 1 drives the internal bus, intended for a low-capacitance node - Side 2 drives the external bus, can withstand stronger ESD and short circuit events"
- note removed: "Receives power and control commands from the host Includes pull-ups in case the I2C interface is not in use"
- moved on the sheet: C1, C2, J1, J3, R1, R2, U2
