File: hardware/v0.2/span.kicad_sch (KiCad schematic)
At the start: 10 parts, among them J10 S4B-XH-A, U7 DRV8434SPWPR

Commit message: Finalize for production
Parts:
- J10: FT Rotation Offset (none) -> 180; LCSC (none) -> C157925
Changed lines of the file:
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@@
+			)
+		)
+		(property "LCSC" "C157925"
+			(at 209.55 96.52 0)
+			(effects
+				(font
+					(size 1.27 1.27)
+				)
+				(hide yes)
+			)
+		)
+		(property "FT Rotation Offset" "180"
+			(at 209.55 96.52 0)
+			(effects
+				(font
+					(size 1.27 1.27)
+				)
+				(hide yes)
 			)
 		)
