File: hardware/v0.3/bed-lift.kicad_sch (KiCad schematic)
At the start: 43 parts, among them J1 SM04B-SRSS-TB, J2 S2P-VH, J3 SM04B-SRSS-TB, J4 TC2030-NL, J5 PH1-06-UA, J6 S3B-XH-A, J7 S6B-XH-A, U1 LP2985-33DBVR, U2 ISO1640, U3 STM32C031K6T6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

Commit message: Update v0.3 to address errata.
Moved the board design and errata into a versioned documents.
Added some photos of the bed.
Connections:
- net ~{DRV_SLEEP}: now also U3.3 (PC15); no longer U3.10 (PA3)
- net ~{SPAN_FAULT}: now also U3.10 (PA3); no longer U3.11 (PA4)
- new net SPI1_NSS: U3.11 (PA4)
- no-connect marks 5 -> 4
Other:
- sheet span1 ports: added ~{SCS}; removed none
- sheet span2 ports: added ~{SCS}; removed none
- sheet span3 ports: added ~{SCS}; removed none
- sheet span4 ports: added ~{SCS}; removed none
- moved on the sheet: C14, R16, U4
