File: hardware/v0.3/span.kicad_sch (KiCad schematic)
At the start: 10 parts, among them J10 S4B-XH-A, U7 DRV8434SPWPR

Commit message: Update v0.3 to address errata.
Moved the board design and errata into a versioned documents.
Added some photos of the bed.
Connections:
- net GND: no longer U7.18 (~{SCS})
- new net ~{SCS}: U7.18 (~{SCS})
Other:
- note added: "Device controlled over SPI so STEP and DIR not used VREF tied to DVDD for full-scale current limit, can be scaled down with TRQ_DAC register"
- note removed: "Device controlled over SPI so STEP and DIR not used ~{SCS} pulled low assuming this is the only device on the SPI bus VREF tied to DVDD for full-scale current limit, can be scaled down with TRQ_DAC register"
Changed lines of the file:
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@@
 		)
 	)
-	(text "Device controlled over SPI so STEP and DIR not used\n~{SCS} pulled low assuming this is the only device on the SPI bus\nVREF tied to DVDD for full-scale current limit, can be scaled\n	down with TRQ_DAC register"
+	(text "Device controlled over SPI so STEP and DIR not used\nVREF tied to DVDD for full-scale current limit, can be scaled\n	down with TRQ_DAC register"
 		(exclude_from_sim no)
-		(at 59.69 125.73 0)
+		(at 59.69 127 0)
 		(effects
 			(font
@@
 		(shape output)
 		(at 146.05 100.33 180)
+		(effects
+			(font
+				(size 1.27 1.27)
+			)
+			(justify right)
+		)
+	)
+	(hierarchical_label "~{SCS}"
+		(shape input)
+		(at 146.05 105.41 180)
 		(effects
 			(font
@@
 				(justify left)
 				(hide yes)
-			)
-		)
-	)
-	(symbol
-		(lib_id "power:GND")
-		(at 146.05 105.41 270)
-		(mirror x)
-		(unit 1)
-		(exclude_from_sim no)
-		(in_bom yes)
-		(on_board yes)
-		(dnp no)
-		(fields_autoplaced yes)
-		(property "Reference" "#PWR046"
-			(at 139.7 105.41 0)
-			(effects
-				(font
-					(size 1.27 1.27)
-				)
-				(hide yes)
-			)
-		)
-		(property "Value" "GND"
-			(at 142.8751 105.41 90)
-			(effects
-				(font
-					(size 1.27 1.27)
-				)
-				(justify right)
-			)
-		)
-		(property "Footprint" ""
-			(at 146.05 105.41 0)
-			(effects
-				(font
-					(size 1.27 1.27)
-				)
-				(hide yes)
-			)
-		)
-		(property "Datasheet" ""
-			(at 146.05 105.41 0)
-			(effects
-				(font
-					(size 1.27 1.27)
-				)
-				(hide yes)
-			)
-		)
-		(property "Description" "Power symbol creates a global label with name \"GND\" , ground"
-			(at 146.05 105.41 0)
-			(effects
-				(font
-					(size 1.27 1.27)
-				)
-				(hide yes)
-			)
-		)
-		(pin "1"
-		)
-		(instances
-			(project "bed-lift"
-				(path "/e474b45c-bd68-4fa4-b324-364b1493394e/442ee682-ada2-425f-9798-dd2a09ab0c93"
-					(reference "#PWR057")
-					(unit 1)
-				)
-				(path "/e474b45c-bd68-4fa4-b324-364b1493394e/7263d767-1c81-4e55-be7f-df3742b1a336"
-					(reference "#PWR068")
-					(unit 1)
-				)
-				(path "/e474b45c-bd68-4fa4-b324-364b1493394e/78bb3d31-b385-4c21-be56-600b0b690b74"
-					(reference "#PWR046")
-					(unit 1)
-				)
-				(path "/e474b45c-bd68-4fa4-b324-364b1493394e/bd85a680-67bc-44d2-872a-bfd1d0a269a3"
-					(reference "#PWR079")
-					(unit 1)
-				)
 			)
 		)
@@
 			(project "bed-lift"
 				(path "/e474b45c-bd68-4fa4-b324-364b1493394e/442ee682-ada2-425f-9798-dd2a09ab0c93"
-					(reference "#PWR055")
+					(reference "#PWR054")
 					(unit 1)
 				)
 				(path "/e474b45c-bd68-4fa4-b324-364b1493394e/7263d767-1c81-4e55-be7f-df3742b1a336"
-					(reference "#PWR066")
+					(reference "#PWR064")
 					(unit 1)
 				)
@@
 				)
 				(path "/e474b45c-bd68-4fa4-b324-364b1493394e/bd85a680-67bc-44d2-872a-bfd1d0a269a3"
-					(reference "#PWR077")
+					(reference "#PWR074")
 					(unit 1)
 				)
@@
 		(dnp no)
 		(fields_autoplaced yes)
-		(property "Reference" "#PWR051"
+		(property "Reference" "#PWR050"
 			(at 146.05 133.35 0)
 			(effects
@@
 			(project "bed-lift"
 				(path "/e474b45c-bd68-4fa4-b324-364b1493394e/442ee682-ada2-425f-9798-dd2a09ab0c93"
-					(reference "#PWR062")
+					(reference "#PWR060")
 					(unit 1)
 				)
 				(path "/e474b45c-bd68-4fa4-b324-364b1493394e/7263d767-1c81-4e55-be7f-df3742b1a336"
-					(reference "#PWR073")
+					(reference "#PWR070")
 					(unit 1)
 				)
 				(path "/e474b45c-bd68-4fa4-b324-364b1493394e/78bb3d31-b385-4c21-be56-600b0b690b74"
-					(reference "#PWR051")
+					(reference "#PWR050")
 					(unit 1)
 				)
 				(path "/e474b45c-bd68-4fa4-b324-364b1493394e/bd85a680-67bc-44d2-872a-bfd1d0a269a3"
-					(reference "#PWR084")
+					(reference "#PWR080")
 					(unit 1)
 				)
@@
 		(dnp no)
 		(fields_autoplaced yes)
-		(property "Reference" "#PWR047"
+		(property "Reference" "#PWR046"
 			(at 198.12 110.49 0)
 			(effects
@@
 			(project "bed-lift"
 				(path "/e474b45c-bd68-4fa4-b324-364b1493394e/442ee682-ada2-425f-9798-dd2a09ab0c93"
-					(reference "#PWR058")
+					(reference "#PWR056")
 					(unit 1)
 				)
 				(path "/e474b45c-bd68-4fa4-b324-364b1493394e/7263d767-1c81-4e55-be7f-df3742b1a336"
-					(reference "#PWR069")
+					(reference "#PWR066")
 					(unit 1)
 				)
 				(path "/e474b45c-bd68-4fa4-b324-364b1493394e/78bb3d31-b385-4c21-be56-600b0b690b74"
-					(reference "#PWR047")
+					(reference "#PWR046")
 					(unit 1)
 				)
 				(path "/e474b45c-bd68-4fa4-b324-364b1493394e/bd85a680-67bc-44d2-872a-bfd1d0a269a3"
-					(reference "#PWR080")
+					(reference "#PWR076")
 					(unit 1)
 				)
@@
 			(project "bed-lift"
 				(path "/e474b45c-bd68-4fa4-b324-364b1493394e/442ee682-ada2-425f-9798-dd2a09ab0c93"
-					(reference "#PWR052")
+					(reference "#PWR051")
 					(unit 1)
 				)
 				(path "/e474b45c-bd68-4fa4-b324-364b1493394e/7263d767-1c81-4e55-be7f-df3742b1a336"
-					(reference "#PWR063")
+					(reference "#PWR061")
 					(unit 1)
 				)
@@
 				)
 				(path "/e474b45c-bd68-4fa4-b324-364b1493394e/bd85a680-67bc-44d2-872a-bfd1d0a269a3"
-					(reference "#PWR074")
+					(reference "#PWR071")
 					(unit 1)
 				)
@@
 			(project "bed-lift"
 				(path "/e474b45c-bd68-4fa4-b324-364b1493394e/442ee682-ada2-425f-9798-dd2a09ab0c93"
-					(reference "#PWR053")
+					(reference "#PWR052")
 					(unit 1)
 				)
 				(path "/e474b45c-bd68-4fa4-b324-364b1493394e/7263d767-1c81-4e55-be7f-df3742b1a336"
-					(reference "#PWR064")
+					(reference "#PWR062")
 					(unit 1)
 				)
@@
 				)
 				(path "/e474b45c-bd68-4fa4-b324-364b1493394e/bd85a680-67bc-44d2-872a-bfd1d0a269a3"
-					(reference "#PWR075")
+					(reference "#PWR072")
 					(unit 1)
 				)
@@
 		(dnp no)
 		(fields_autoplaced yes)
-		(property "Reference" "#PWR048"
+		(property "Reference" "#PWR047"
 			(at 198.12 113.03 0)
 			(effects
@@
 			(project "bed-lift"
 				(path "/e474b45c-bd68-4fa4-b324-364b1493394e/442ee682-ada2-425f-9798-dd2a09ab0c93"
-					(reference "#PWR059")
+					(reference "#PWR057")
 					(unit 1)
 				)
 				(path "/e474b45c-bd68-4fa4-b324-364b1493394e/7263d767-1c81-4e55-be7f-df3742b1a336"
-					(reference "#PWR070")
+					(reference "#PWR067")
 					(unit 1)
 				)
 				(path "/e474b45c-bd68-4fa4-b324-364b1493394e/78bb3d31-b385-4c21-be56-600b0b690b74"
-					(reference "#PWR048")
+					(reference "#PWR047")
 					(unit 1)
 				)
 				(path "/e474b45c-bd68-4fa4-b324-364b1493394e/bd85a680-67bc-44d2-872a-bfd1d0a269a3"
-					(reference "#PWR081")
+					(reference "#PWR077")
 					(unit 1)
 				)
@@
 			(project "bed-lift"
 				(path "/e474b45c-bd68-4fa4-b324-364b1493394e/442ee682-ada2-425f-9798-dd2a09ab0c93"
-					(reference "#PWR056")
+					(reference "#PWR055")
 					(unit 1)
 				)
 				(path "/e474b45c-bd68-4fa4-b324-364b1493394e/7263d767-1c81-4e55-be7f-df3742b1a336"
-					(reference "#PWR067")
+					(reference "#PWR065")
 					(unit 1)
 				)
@@
 				)
 				(path "/e474b45c-bd68-4fa4-b324-364b1493394e/bd85a680-67bc-44d2-872a-bfd1d0a269a3"
-					(reference "#PWR078")
+					(reference "#PWR075")
 					(unit 1)
 				)
@@
 		(dnp no)
 		(fields_autoplaced yes)
-		(property "Reference" "#PWR050"
+		(property "Reference" "#PWR049"
 			(at 198.12 115.57 0)
 			(effects
@@
 			(project "bed-lift"
 				(path "/e474b45c-bd68-4fa4-b324-364b1493394e/442ee682-ada2-425f-9798-dd2a09ab0c93"
-					(reference "#PWR061")
+					(reference "#PWR059")
 					(unit 1)
 				)
 				(path "/e474b45c-bd68-4fa4-b324-364b1493394e/7263d767-1c81-4e55-be7f-df3742b1a336"
-					(reference "#PWR072")
+					(reference "#PWR069")
 					(unit 1)
 				)
 				(path "/e474b45c-bd68-4fa4-b324-364b1493394e/78bb3d31-b385-4c21-be56-600b0b690b74"
-					(reference "#PWR050")
+					(reference "#PWR049")
 					(unit 1)
 				)
 				(path "/e474b45c-bd68-4fa4-b324-364b1493394e/bd85a680-67bc-44d2-872a-bfd1d0a269a3"
-					(reference "#PWR083")
+					(reference "#PWR079")
 					(unit 1)
 				)
@@
 		(on_board yes)
 		(dnp no)
-		(property "Reference" "#PWR049"
+		(property "Reference" "#PWR048"
 			(at 140.97 115.57 0)
 			(effects
@@
 			(project "bed-lift"
 				(path "/e474b45c-bd68-4fa4-b324-364b1493394e/442ee682-ada2-425f-9798-dd2a09ab0c93"
-					(reference "#PWR060")
+					(reference "#PWR058")
 					(unit 1)
 				)
 				(path "/e474b45c-bd68-4fa4-b324-364b1493394e/7263d767-1c81-4e55-be7f-df3742b1a336"
-					(reference "#PWR071")
+					(reference "#PWR068")
 					(unit 1)
 				)
 				(path "/e474b45c-bd68-4fa4-b324-364b1493394e/78bb3d31-b385-4c21-be56-600b0b690b74"
-					(reference "#PWR049")
+					(reference "#PWR048")
 					(unit 1)
 				)
 				(path "/e474b45c-bd68-4fa4-b324-364b1493394e/bd85a680-67bc-44d2-872a-bfd1d0a269a3"
-					(reference "#PWR082")
+					(reference "#PWR078")
 					(unit 1)
 				)
@@
 			(project "bed-lift"
 				(path "/e474b45c-bd68-4fa4-b324-364b1493394e/442ee682-ada2-425f-9798-dd2a09ab0c93"
-					(reference "#PWR054")
+					(reference "#PWR053")
 					(unit 1)
 				)
 				(path "/e474b45c-bd68-4fa4-b324-364b1493394e/7263d767-1c81-4e55-be7f-df3742b1a336"
-					(reference "#PWR065")
+					(reference "#PWR063")
 					(unit 1)
 				)
@@
 				)
 				(path "/e474b45c-bd68-4fa4-b324-364b1493394e/bd85a680-67bc-44d2-872a-bfd1d0a269a3"
-					(reference "#PWR076")
-					(unit 1)
-				)
+					(reference "#PWR073")
+					(unit 1)
+				)
