File: hardware/v1.0/bed-lift.kicad_pcb (KiCad board)
At the start: 4 copper layers, 195 x 45 mm, 143 parts, among them J1 SM04B-SRSS-TB, J10 Molex Mini Fit Jr 39-30-1060, J11 S4B-XH-A, J12 S4B-XH-A, J13 S4B-XH-A, J14 S4B-XH-A, J2 S2P-VH, J3 SM04B-SRSS-TB, J4 S3B-XH-A, J5 S6B-XH-A, J6 Conn_ST_STDC14, J7 S6B-XH-A, J8 Conn_02x08_Odd_Even, J9 Molex Mini Fit Jr 39-30-1060, Q1 MMBT3904, U1 LP2985-33DBVR, U10 DRV8434SPWPR, U2 LP2985-5.0DBVR, U3 ISO1640, U4 STM32C051C8T6, U5 DRV8874PWPR, U6 DRV8874PWPR, U7 DRV8434SPWPR, U8 DRV8434SPWPR, U9 DRV8434SPWPR

Commit message: Further refinement.
Parts:
- added C10: 1u, Capacitor_SMD:C_0603_1608Metric, F.Cu at (90.2, 86.0)
- added C23: 100n, Capacitor_SMD:C_0402_1005Metric, F.Cu at (112.0, 71.2)
- added C26: 1u, Capacitor_SMD:C_0603_1608Metric, F.Cu at (111.8, 76.8)
- added C33: 100n, Capacitor_SMD:C_0402_1005Metric, F.Cu at (136.0, 71.2)
- added C36: 1u, Capacitor_SMD:C_0603_1608Metric, F.Cu at (135.8, 76.8)
- added D4: KT-0603R, LED_SMD:LED_0603_1608Metric, F.Cu at (61.5, 63.0)
- added D5: PESD3V3L5UY, Package_TO_SOT_SMD:SOT-363_SC-70-6, F.Cu at (46.0, 66.0)
- added J8: BM04B-SRSS-TB, Connector_JST:JST_SH_BM04B-SRSS-TB_1x04-1MP_P1.00mm_Vertical, F.Cu at (41.8, 57.8)
- added R29: 1K, Resistor_SMD:R_0402_1005Metric, F.Cu at (62.0, 64.5)
- C1, C13, C14, C2, C5, C8: footprint Capacitor_SMD:C_0603_1608Metric -> Capacitor_SMD:C_0402_1005Metric
- C15: renamed from C12; footprint Capacitor_SMD:C_0603_1608Metric -> Capacitor_SMD:C_0402_1005Metric
- C16: renamed from C15; footprint Capacitor_SMD:C_0603_1608Metric -> Capacitor_SMD:C_0402_1005Metric
- C17: renamed from C16; footprint Capacitor_SMD:C_0603_1608Metric -> Capacitor_SMD:C_0402_1005Metric
- C24: renamed from C22; footprint Capacitor_SMD:C_0603_1608Metric -> Capacitor_SMD:C_0402_1005Metric
- C25: renamed from C23; footprint Capacitor_SMD:C_0603_1608Metric -> Capacitor_SMD:C_0402_1005Metric
- C27: renamed from C24; footprint Capacitor_SMD:C_0603_1608Metric -> Capacitor_SMD:C_0402_1005Metric
- C34: renamed from C30; footprint Capacitor_SMD:C_0603_1608Metric -> Capacitor_SMD:C_0402_1005Metric
- C35: renamed from C31; footprint Capacitor_SMD:C_0603_1608Metric -> Capacitor_SMD:C_0402_1005Metric
- C37: renamed from C32; footprint Capacitor_SMD:C_0603_1608Metric -> Capacitor_SMD:C_0402_1005Metric
- R1, R10, R11, R12, R13, R14, R15, R16, R17, R2, R20, R21, R23, R24, R25, R26, R27, R28, R3, R4, R5, R6, R7, R8, R9: footprint Resistor_SMD:R_0603_1608Metric -> Resistor_SMD:R_0402_1005Metric
- R18: renamed from R29; footprint Resistor_SMD:R_0603_1608Metric -> Resistor_SMD:R_0402_1005Metric
- R19: renamed from R30; footprint Resistor_SMD:R_0603_1608Metric -> Resistor_SMD:R_0402_1005Metric
- R22: value 1K -> 3.3K
- R30: renamed from R18; footprint Resistor_SMD:R_0603_1608Metric -> Resistor_SMD:R_0402_1005Metric
- R31: renamed from R19; footprint Resistor_SMD:R_0603_1608Metric -> Resistor_SMD:R_0402_1005Metric
- R32: renamed from R31; footprint Resistor_SMD:R_0603_1608Metric -> Resistor_SMD:R_0402_1005Metric
- R33: renamed from R32; footprint Resistor_SMD:R_0603_1608Metric -> Resistor_SMD:R_0402_1005Metric
- R34: renamed from R33; footprint Resistor_SMD:R_0603_1608Metric -> Resistor_SMD:R_0402_1005Metric
- R35: renamed from R34; footprint Resistor_SMD:R_0603_1608Metric -> Resistor_SMD:R_0402_1005Metric
- R36: renamed from R35; footprint Resistor_SMD:R_0603_1608Metric -> Resistor_SMD:R_0402_1005Metric
- R37: renamed from R36; footprint Resistor_SMD:R_0603_1608Metric -> Resistor_SMD:R_0402_1005Metric
- U2: value LP2985-5.0DBVR -> LP2985-50DBVR
- moved R19 18.0 mm to (50.6, 58.2), turned to 90 degrees
- moved R18 13.3 mm to (52.0, 58.2), turned to 90 degrees
- moved R6 5.34 mm to (68.2, 86.0)
- moved J6 5.00 mm to (72.9, 59.8)
- moved R31 4.78 mm to (43.2, 64.5)
- moved R21 4.61 mm to (43.5, 86.0)
- moved R20 3.64 mm to (48.5, 86.0)
- moved R17 3.16 mm to (79.2, 86.0)
- moved R7 2.93 mm to (63.2, 86.0)
- moved R11 2.69 mm to (80.5, 86.0)
- moved R13 2.24 mm to (62.0, 86.0)
- moved R23 2.24 mm to (55.8, 86.0)
- moved R8 2.02 mm to (88.0, 86.0)
- moved R16 1.91 mm to (81.8, 86.0)
- moved R3 1.90 mm to (82.8, 78.5)
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- renumbered C10 to C11, C11 to C12, C17 to C18, C18 to C19, C19 to C20, C20 to C21, C21 to C22, C25 to C28, C26 to C29, C27 to C30, C28 to C31, C29 to C32, C33 to C38, C34 to C39, C35 to C40, C36 to C41, C37 to C42, C38 to C43, C39 to C44, C40 to C45, C41 to C46, C42 to C47, C43 to C48, C44 to C49, C45 to C50, C46 to C51, C47 to C52, C48 to C53, C49 to C54, C50 to C55, C51 to C56, C52 to C57, C53 to C58, C54 to C59, C55 to C60, C56 to C61, C57 to C62, C58 to C63, C59 to C64, C60 to C65, C61 to C66, C62 to C67, C63 to C68, C64 to C69, J9 to J10, J10 to J11, J11 to J12, J12 to J13, J13 to J14, J14 to J15, J8 to J6, J6 to J9
Connections:
- net /LED_B renamed /LED_STATUS_B
- net /LED_G renamed /LED_STATUS_G
- net /LED_R renamed /LED_STATUS_R
- J1 pad MP: unconnected-(J1-MountPin-PadMP)_1 -> /BUS_GND
- J3 pad MP: unconnected-(J3-MountPin-PadMP) -> /BUS_GND
- J6 pad 12: /EXP_PA8 -> /EXP_PA12
- J6 pad 14: /EXP_PA12 -> unconnected-(J6-Pin_14-Pad14)
- U4 pad 28: /EXP_PA8 -> /~{LED_POWER}
Routing:
- net /INT_I2C_SDA: track 12.1 -> 34.3 mm, vias 0 -> 1
- net +3.3V: track 356.2 -> 377.9 mm, vias 15 -> 18
- net /INT_I2C_SCL: track 19.6 -> 38.2 mm, vias 0 -> 1
- net /EXP_PA8: track 12.6 -> 0.00 mm
- net /~{SPAN1_LIMIT_A}: track 40.1 -> 44.6 mm
- net Net-(J7-Pin_3): track 11.2 -> 7.23 mm
- net /~{SPAN1_LIMIT_B}: track 42.3 -> 46.3 mm
- net Net-(J7-Pin_2): track 10.7 -> 6.98 mm
- net /EXP_PA12: track 13.1 -> 9.88 mm
- net +5V: track 141.0 -> 138.1 mm
- net Net-(J4-Pin_3): track 10.8 -> 7.99 mm
- net /~{SPAN2_LIMIT_A}: track 43.1 -> 45.8 mm
- net Net-(J4-Pin_2): track 10.4 -> 7.75 mm
- net /~{LED_POWER}: track 0.00 -> 2.40 mm
- net Net-(J10-Pin_1): track 22.5 -> 24.8 mm
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- added copper zone on F.Cu, net /BUS_GND
- added copper zone on In1.Cu, net /BUS_GND
Other:
- board text added: "BT0 (NC) PA12 PB12 SCL 3V3 5V 12V"
- board text added: "EXT I2C"
- board text added: "INT I2C"
- board text added: "POWER"
- board text removed: "BT0 PA12 PA8 PB12 SCL 3V3 5V 12V"
- board text removed: "QWIIC"
