File: hardware/v1.0/bed-lift.kicad_sch (KiCad schematic)
At the start: 64 parts, among them J1 SM04B-SRSS-TB, J2 S2P-VH, J3 SM04B-SRSS-TB, J4 S3B-XH-A, J5 S6B-XH-A, J6 Conn_ST_STDC14, J7 S6B-XH-A, J8 Conn_02x08_Odd_Even, Q1 MMBT3904, U1 LP2985-33DBVR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

Commit message: Further refinement, ready for fabrication.
Parts:
- added C10: 1u, Capacitor_SMD:C_0603_1608Metric, symbol Device:C
- added D4: KT-0603R, LED_SMD:LED_0603_1608Metric, symbol Device:LED
- added D5: PESD3V3L5UY, Package_TO_SOT_SMD:SOT-363_SC-70-6, symbol Power_Protection:PESD3V3L5UY
- added J8: BM04B-SRSS-TB, Connector_JST:JST_SH_BM04B-SRSS-TB_1x04-1MP_P1.00mm_Vertical, symbol Connector_Generic_MountingPin:Conn_01x04_MountingPin
- added R29: 2.2K, Resistor_SMD:R_0402_1005Metric, symbol Device:R
- C1, C13, C14, C2: footprint Capacitor_SMD:C_0603_1608Metric -> Capacitor_SMD:C_0402_1005Metric; LCSC C14663 -> C1525; Rating 50V, X7R -> 16V, X7R
- C15: renamed from C12; footprint Capacitor_SMD:C_0603_1608Metric -> Capacitor_SMD:C_0402_1005Metric; LCSC C14663 -> C1525; Rating 50V, X7R -> 16V, X7R
- C16: renamed from C15; footprint Capacitor_SMD:C_0603_1608Metric -> Capacitor_SMD:C_0402_1005Metric; LCSC C14663 -> C1525; Rating 50V, X7R -> 16V, X7R
- C17: renamed from C16; footprint Capacitor_SMD:C_0603_1608Metric -> Capacitor_SMD:C_0402_1005Metric; LCSC C14663 -> C1525; Rating 50V, X7R -> 16V, X7R
- C5, C8: footprint Capacitor_SMD:C_0603_1608Metric -> Capacitor_SMD:C_0402_1005Metric; LCSC C57112 -> C15195
- J1, J3: Label EXT QWIIC -> EXT I2C
- R1, R12, R13, R14, R15, R16, R17, R2, R26, R28: footprint Resistor_SMD:R_0603_1608Metric -> Resistor_SMD:R_0402_1005Metric; LCSC C4190 -> C25879
- R10, R11, R20, R21, R6, R7, R8, R9: footprint Resistor_SMD:R_0603_1608Metric -> Resistor_SMD:R_0402_1005Metric; LCSC C31850 -> C25768
- R18: renamed from R29; footprint Resistor_SMD:R_0603_1608Metric -> Resistor_SMD:R_0402_1005Metric; LCSC C4190 -> C25879
- R19: renamed from R30; footprint Resistor_SMD:R_0603_1608Metric -> Resistor_SMD:R_0402_1005Metric; LCSC C4190 -> C25879
- R22: value 1K -> 3.3K; LCSC C21190 -> C22978
- R23, R24, R25: footprint Resistor_SMD:R_0603_1608Metric -> Resistor_SMD:R_0402_1005Metric; LCSC C22962 -> C25091
- R27, R3, R4, R5: footprint Resistor_SMD:R_0603_1608Metric -> Resistor_SMD:R_0402_1005Metric; LCSC C25804 -> C25744
- R30: renamed from R18; footprint Resistor_SMD:R_0603_1608Metric -> Resistor_SMD:R_0402_1005Metric; LCSC C25803 -> C25741
- R31: renamed from R19; footprint Resistor_SMD:R_0603_1608Metric -> Resistor_SMD:R_0402_1005Metric; LCSC C25803 -> C25741
- U2: value LP2985-5.0DBVR -> LP2985-50DBVR
- renumbered C10 to C11, C11 to C12, J8 to J6, J6 to J9
Connections:
- net +3.3V: now also D4.2 (A), J8.2 (Pin_2)
- net +5V: now also C10.1
- net BUS_GND: now also J1.MP (MountPin), J3.MP (MountPin)
- net CONSOLE_RX: now also D5.3 (K2)
- net CONSOLE_TX: now also D5.1 (K1)
- net EXP_PA12: now also J6.12 (Pin_12); no longer J6.14 (Pin_14)
- net GND: now also C10.2, D5.2 (A), J8.1 (Pin_1), J8.MP (MountPin)
- net INT_I2C_SCL: now also J8.4 (Pin_4)
- net INT_I2C_SDA: now also J8.3 (Pin_3)
- net SWCLK/BOOT0: now also D5.5 (K4)
- net SWDIO: now also D5.6 (K5)
- net ~{RESET}: now also D5.4 (K3)
- net EXP_PA8 renamed ~{LED_POWER}
- net ~{LED_POWER}: now also R29.2; no longer J6.12 (Pin_12)
- net LED_B renamed LED_STATUS_B
- net LED_G renamed LED_STATUS_G
- net LED_R renamed LED_STATUS_R
- new net: D4.1 (K), R29.1
- no-connect marks 6 -> 5
Other:
- note added: "Debounce switch contacts, ESD protection Control indicators rated for 15 mA at 3 V"
- note added: "EXTERNAL I2C INTERFACE (QWIIC)"
- note added: "Programmed via SWD with STLINK-V3 and an STDC14 cable Can also access the system bootloader over I2C or UART by pulling BOOT0 low during RESET Unused pins are exposed via an expansion port including an internal I2C interface (QWIIC)"
- note removed: "EXTERNAL QWIIC INTERFACE"
- note removed: "Programmed via SWD with STLINK-V3 and an STDC14 cable Can also access the system bootloader over I2C or UART by pulling BOOT0 low during RESET Unused pins are exposed via an expansion port including an internal I2C port"
- moved on the sheet: C11, C12, C15, J5, J6, J9, R18, R19, R30, R31
