File: hardware/v1.0/lift.kicad_sch (KiCad schematic)
At the start: 13 parts, among them J9 Molex Mini Fit Jr 39-30-1060, U5 DRV8874PWPR

Commit message: Further refinement, ready for fabrication.
Parts:
- added C23: 100n, Capacitor_SMD:C_0402_1005Metric, symbol Device:C
- added C26: 1u, Capacitor_SMD:C_0603_1608Metric, symbol Device:C
- added D6: PESD5V0S2UAT, Package_TO_SOT_SMD:SOT-23, symbol Device:D_Zener_Dual_CommonAnode_KKA_Parallel
- C24: renamed from C22; footprint Capacitor_SMD:C_0603_1608Metric -> Capacitor_SMD:C_0402_1005Metric; LCSC C57112 -> C15195
- C25: renamed from C23; footprint Capacitor_SMD:C_0603_1608Metric -> Capacitor_SMD:C_0402_1005Metric; LCSC C57112 -> C15195
- C27: renamed from C24; footprint Capacitor_SMD:C_0603_1608Metric -> Capacitor_SMD:C_0402_1005Metric; LCSC C57112 -> C15195
- R32: renamed from R31; footprint Resistor_SMD:R_0603_1608Metric -> Resistor_SMD:R_0402_1005Metric; LCSC C21190 -> C11702
- R33: renamed from R32; footprint Resistor_SMD:R_0603_1608Metric -> Resistor_SMD:R_0402_1005Metric; LCSC C21190 -> C11702
- R34: renamed from R33; footprint Resistor_SMD:R_0603_1608Metric -> Resistor_SMD:R_0402_1005Metric; LCSC C23179 -> C25117
- renumbered C17 to C18, C18 to C19, C19 to C20, C20 to C21, C21 to C22, J9 to J10
Connections:
- net +3.3V: now also C23.1
- net +5V: now also C26.1
- net GND: now also C23.2, C26.2, D6.3 (A)
- net at J10.1 (Pin_1), R32.2: now also D6.2 (K)
- net at J10.6 (Pin_6), R33.1: now also D6.1 (K)
Other:
- note added: "The hall sensor outputs are push-pull at 5 V, RC filter cutoff at 15.9 kHz"
- note removed: "The hall sensor outputs are push-pull at 5 V, RC filter for jitter"
- moved on the sheet: C24, C25, C27, R32, R33, R34
