File: hardware/v1.0/lift.kicad_sch (KiCad schematic)
At the start: 13 parts, among them J8 Molex Mini Fit Jr 39-30-1060, U5 DRV8874PWPR

Commit message: Complete first draft of v1.0 hardware.
Parts:
- removed C16: 10u, Capacitor_SMD:C_0805_2012Metric, symbol Device:C
- removed C20, C21: 10n, Capacitor_SMD:C_0603_1608Metric, symbol Device:C
- removed NT2: NetTie_2, Generic:NetTie-2_SMD_Pad2.5mm, symbol Device:NetTie_2
- added C17: 47u, Capacitor_THT:CP_Radial_D5.0mm_P2.50mm, symbol Device:C_Polarized
- added C18: 22u, Capacitor_SMD:C_1210_3225Metric, symbol Device:C
- added C23, C24: 10n, Capacitor_SMD:C_0603_1608Metric, symbol Device:C
- C19: renamed from C17; Rating 50V, X5R -> 50V, X7R
- C20: renamed from C18; Rating 50V, X5R -> 50V, X7R
- C21: renamed from C19; Rating 50V, X5R -> 50V, X7R
- C22: renamed from C15; Rating 50V, X5R -> 50V, X7R
- renumbered J8 to J9, R18 to R31, R19 to R32, R17 to R33
Connections:
- net VM is gone; now on net +12V: C19.1, C20.1, U5.11 (VM)
- net +12V: now also C17.1, C18.2
- net GND: now also C17.2, C18.1, C23.2, C24.2
- net HALL1: now also C24.1
- net HALL2: now also C23.1
- net EXT_HALL1: no longer names the net of J9.6 (Pin_6), R32.1
- net EXT_HALL2: no longer names the net of J9.1 (Pin_1), R31.2
Other:
- note added: "Designed for 12 V DC motor load up to 3 A (driver is rated for 6 A peak)"
- note added: "LIFT ACTUATOR MOTOR DRIVER"
- note added: "PMODE set to use PWM mode via IN1 and IN2 IMODE set to fixed off-time current chopping, outputs latched off overcurrent response ~{SLEEP} enables driver when high ~{FAULT} is open-drain"
- note added: "The hall sensor outputs are push-pull at 5 V, RC filter for jitter"
- note removed: "BED PLATFORM LIFT MOTOR DRIVER"
- note removed: "Designed for 12 V DC motor load up to 3 A (6 A peak)"
- note removed: "PMODE set to use PWM mode IMODE set to fixed off-time current chopping, outputs latched off overcurrent response ~{SLEEP} enables driver when high ~{FAULT} is open-drain Internal pull-down on ~{SLEEP}, IN1, and IN2 keeps motor off until MCU is initialized"
- moved on the sheet: C19, C20, C21, C22, J9, R31, R32, R33, U5

Commit message: Improve power distribution.
Connections:
- net VHALL renamed +5V
Changed lines of the file:
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@@
 	(title_block
 		(title "Bed Lift Controller")
-		(date "2025-10")
-		(rev "v0.2.1")
+		(date "2026-01")
+		(rev "v1.0")
 		(company "Brown Studios LLC")
+		(comment 1 "github.com/j9brown/bed-lift")
 	)
 	(rectangle
@@
 		(shape input)
 		(at 157.48 68.58 180)
-		(effects
-			(font
-				(size 1.27 1.27)
-			)
-			(justify right)
-		)
-	)
-	(hierarchical_label "VHALL"
-		(shape passive)
-		(at 151.13 124.46 180)
 		(effects
 			(font
@@
 		(length 2.54)
 		(shape round)
-		(at 153.67 124.46 0)
-		(fields_autoplaced yes)
-		(effects
-			(font
-				(size 1.27 1.27)
-			)
-			(justify left bottom)
-		)
-		(property "Netclass" "Power"
-			(at 154.3685 121.92 0)
-			(effects
-				(font
-					(size 1.27 1.27)
-					(italic yes)
-				)
-				(justify left)
-				(hide yes)
-			)
-		)
-	)
-	(netclass_flag ""
-		(length 2.54)
-		(shape round)
 		(at 160.02 55.88 0)
 		(fields_autoplaced yes)
@@
 				(justify left)
 				(hide yes)
+			)
+		)
+	)
+	(symbol
+		(lib_id "power:+5V")
+		(at 151.13 124.46 90)
+		(unit 1)
+		(exclude_from_sim no)
+		(in_bom yes)
+		(on_board yes)
+		(dnp no)
+		(fields_autoplaced yes)
+		(property "Reference" "#PWR045"
+			(at 154.94 124.46 0)
+			(effects
+				(font
+					(size 1.27 1.27)
+				)
+				(hide yes)
+			)
+		)
+		(property "Value" "+5V"
+			(at 147.9551 124.46 90)
+			(effects
+				(font
+					(size 1.27 1.27)
+				)
+				(justify left)
+			)
+		)
+		(property "Footprint" ""
+			(at 151.13 124.46 0)
+			(effects
+				(font
+					(size 1.27 1.27)
+				)
+				(hide yes)
+			)
+		)
+		(property "Datasheet" ""
+			(at 151.13 124.46 0)
+			(effects
+				(font
+					(size 1.27 1.27)
+				)
+				(hide yes)
+			)
+		)
+		(property "Description" "Power symbol creates a global label with name \"+5V\""
+			(at 151.13 124.46 0)
+			(effects
+				(font
+					(size 1.27 1.27)
+				)
+				(hide yes)
+			)
+		)
+		(pin "1"
+		)
+		(instances
+			(project "bed-lift"
+				(path "/e474b45c-bd68-4fa4-b324-364b1493394e/73779cb4-e276-4cb8-abc0-7835080fddfe"
+					(reference "#PWR045")
+					(unit 1)
+				)
+				(path "/e474b45c-bd68-4fa4-b324-364b1493394e/b7a1b7cc-1f28-44b5-9bcf-53ef9e40d7ff"
+					(reference "#PWR055")
+					(unit 1)
+				)
 			)
 		)
@@
 		(dnp no)
 		(fields_autoplaced yes)
-		(property "Reference" "#PWR044"
+		(property "Reference" "#PWR042"
 			(at 209.55 88.9 0)
 			(effects
@@
 			(project "bed-lift"
 				(path "/e474b45c-bd68-4fa4-b324-364b1493394e/73779cb4-e276-4cb8-abc0-7835080fddfe"
-					(reference "#PWR044")
+					(reference "#PWR042")
 					(unit 1)
 				)
 				(path "/e474b45c-bd68-4fa4-b324-364b1493394e/b7a1b7cc-1f28-44b5-9bcf-53ef9e40d7ff"
-					(reference "#PWR053")
+					(reference "#PWR052")
 					(unit 1)
 				)
@@
 		(dnp no)
 		(fields_autoplaced yes)
-		(property "Reference" "#PWR048"
+		(property "Reference" "#PWR047"
 			(at 173.99 146.05 0)
 			(effects
@@
 			(project "bed-lift"
 				(path "/e474b45c-bd68-4fa4-b324-364b1493394e/73779cb4-e276-4cb8-abc0-7835080fddfe"
-					(reference "#PWR048")
+					(reference "#PWR047")
 					(unit 1)
 				)
@@
 		(dnp no)
 		(fields_autoplaced yes)
-		(property "Reference" "#PWR041"
+		(property "Reference" "#PWR039"
 			(at 105.41 63.5 0)
 			(effects
@@
 			(project "bed-lift"
 				(path "/e474b45c-bd68-4fa4-b324-364b1493394e/73779cb4-e276-4cb8-abc0-7835080fddfe"
-					(reference "#PWR041")
+					(reference "#PWR039")
 					(unit 1)
 				)
 				(path "/e474b45c-bd68-4fa4-b324-364b1493394e/b7a1b7cc-1f28-44b5-9bcf-53ef9e40d7ff"
-					(reference "#PWR050")
+					(reference "#PWR049")
 					(unit 1)
 				)
@@
 		(dnp no)
 		(fields_autoplaced yes)
-		(property "Reference" "#PWR040"
+		(property "Reference" "#PWR038"
 			(at 93.98 45.72 0)
 			(effects
@@
 			(project "bed-lift"
 				(path "/e474b45c-bd68-4fa4-b324-364b1493394e/73779cb4-e276-4cb8-abc0-7835080fddfe"
-					(reference "#PWR040")
+					(reference "#PWR038")
 					(unit 1)
 				)
 				(path "/e474b45c-bd68-4fa4-b324-364b1493394e/b7a1b7cc-1f28-44b5-9bcf-53ef9e40d7ff"
-					(reference "#PWR049")
+					(reference "#PWR048")
 					(unit 1)
 				)
@@
 		(dnp no)
 		(fields_autoplaced yes)
-		(property "Reference" "#PWR047"
+		(property "Reference" "#PWR046"
 			(at 114.3 142.24 0)
 			(effects
@@
 			(project "bed-lift"
 				(path "/e474b45c-bd68-4fa4-b324-364b1493394e/73779cb4-e276-4cb8-abc0-7835080fddfe"
-					(reference "#PWR047")
+					(reference "#PWR046")
 					(unit 1)
 				)
@@
 		(on_board yes)
 		(dnp no)
-		(property "Reference" "#PWR045"
+		(property "Reference" "#PWR043"
 			(at 161.29 91.44 0)
 			(effects
@@
 			(project "bed-lift"
 				(path "/e474b45c-bd68-4fa4-b324-364b1493394e/73779cb4-e276-4cb8-abc0-7835080fddfe"
-					(reference "#PWR045")
+					(reference "#PWR043")
 					(unit 1)
 				)
 				(path "/e474b45c-bd68-4fa4-b324-364b1493394e/b7a1b7cc-1f28-44b5-9bcf-53ef9e40d7ff"
-					(reference "#PWR054")
+					(reference "#PWR053")
 					(unit 1)
 				)
@@
 		(dnp no)
 		(fields_autoplaced yes)
-		(property "Reference" "#PWR046"
+		(property "Reference" "#PWR044"
 			(at 209.55 91.44 0)
 			(effects
@@
 			(project "bed-lift"
 				(path "/e474b45c-bd68-4fa4-b324-364b1493394e/73779cb4-e276-4cb8-abc0-7835080fddfe"
-					(reference "#PWR046")
+					(reference "#PWR044")
 					(unit 1)
 				)
 				(path "/e474b45c-bd68-4fa4-b324-364b1493394e/b7a1b7cc-1f28-44b5-9bcf-53ef9e40d7ff"
-					(reference "#PWR055")
+					(reference "#PWR054")
 					(unit 1)
 				)
@@
 		(dnp no)
 		(fields_autoplaced yes)
-		(property "Reference" "#PWR043"
+		(property "Reference" "#PWR041"
 			(at 209.55 86.36 0)
 			(effects
@@
 			(project "bed-lift"
 				(path "/e474b45c-bd68-4fa4-b324-364b1493394e/73779cb4-e276-4cb8-abc0-7835080fddfe"
-					(reference "#PWR043")
+					(reference "#PWR041")
 					(unit 1)
 				)
 				(path "/e474b45c-bd68-4fa4-b324-364b1493394e/b7a1b7cc-1f28-44b5-9bcf-53ef9e40d7ff"
-					(reference "#PWR052")
+					(reference "#PWR051")
 					(unit 1)
 				)
@@
 		(on_board yes)
 		(dnp no)
-		(property "Reference" "#PWR042"
+		(property "Reference" "#PWR040"
 			(at 161.29 60.96 0)
 			(effects
@@
 			(project "bed-lift"
 				(path "/e474b45c-bd68-4fa4-b324-364b1493394e/73779cb4-e276-4cb8-abc0-7835080fddfe"
-					(reference "#PWR042")
+					(reference "#PWR040")
 					(unit 1)
 				)
 				(path "/e474b45c-bd68-4fa4-b324-364b1493394e/b7a1b7cc-1f28-44b5-9bcf-53ef9e40d7ff"
-					(reference "#PWR051")
-					(unit 1)
-				)
+					(reference "#PWR050")
+					(unit 1)
+				)

Commit message: Further refinement.
Parts:
- added C23: 100n, Capacitor_SMD:C_0402_1005Metric, symbol Device:C
- added C26: 1u, Capacitor_SMD:C_0603_1608Metric, symbol Device:C
- C24: renamed from C22; footprint Capacitor_SMD:C_0603_1608Metric -> Capacitor_SMD:C_0402_1005Metric; LCSC C57112 -> C15195
- C25: renamed from C23; footprint Capacitor_SMD:C_0603_1608Metric -> Capacitor_SMD:C_0402_1005Metric; LCSC C57112 -> C15195
- C27: renamed from C24; footprint Capacitor_SMD:C_0603_1608Metric -> Capacitor_SMD:C_0402_1005Metric; LCSC C57112 -> C15195
- R32: renamed from R31; footprint Resistor_SMD:R_0603_1608Metric -> Resistor_SMD:R_0402_1005Metric; LCSC C21190 -> C11702
- R33: renamed from R32; footprint Resistor_SMD:R_0603_1608Metric -> Resistor_SMD:R_0402_1005Metric; LCSC C21190 -> C11702
- R34: renamed from R33; footprint Resistor_SMD:R_0603_1608Metric -> Resistor_SMD:R_0402_1005Metric; LCSC C23179 -> C25117
- renumbered C17 to C18, C18 to C19, C19 to C20, C20 to C21, C21 to C22, J9 to J10
Connections:
- net +3.3V: now also C23.1
- net +5V: now also C26.1
- net GND: now also C23.2, C26.2
