File: hardware/v1.0/span.kicad_sch (KiCad schematic)
At the start: 10 parts, among them J10 S4B-XH-A, U7 DRV8434SPWPR

Commit message: Complete first draft of v1.0 hardware.
Parts:
- removed C29: 10u, Capacitor_SMD:C_0805_2012Metric, symbol Device:C
- removed NT4: NetTie_2, Generic:NetTie-2_SMD_Pad1.5mm, symbol Device:NetTie_2
- added C33: 47u, Capacitor_THT:CP_Radial_D5.0mm_P2.50mm, symbol Device:C_Polarized
- added C34: 22u, Capacitor_SMD:C_1210_3225Metric, symbol Device:C
- C35: renamed from C30; Rating 50V, X5R -> 50V, X7R
- C36: renamed from C31; Rating 50V, X5R -> 50V, X7R
- C37: renamed from C32; LCSC C1603 -> C21120; Rating 50V, X5R -> 50V, X7R
- C38: renamed from C33; Rating 50V, X5R -> 50V, X7R
- C39: renamed from C34; footprint Capacitor_SMD:C_0603_1608Metric -> Capacitor_SMD:C_0805_2012Metric; LCSC C15849 -> C28323; Rating 50V, X5R -> 50V, X7R
- C40: renamed from C35; Rating 50V, X5R -> 50V, X7R
- renumbered J10 to J11
Connections:
- net VM is gone; now on net +12V: C35.1, C36.1, C37.1, U7.13 (VM), U7.2 (VM)
- net +12V: now also C33.1, C34.2
- net +3.3V: now also U7.17 (VREF)
- net DVDD: no longer U7.17 (VREF)
- net GND: now also C33.2, C34.1; no longer U7.23 (STEP)
- new net STEP: U7.23 (STEP)
Other:
- note added: "Designed for 12 V DC stepper motor load up to 1.8 A rms"
- note added: "SPAN ACTUATOR MOTOR DRIVER"
- note added: "~{SLEEP} enables driver when high ~{FAULT} is open-drain ENABLE has internal pull-up to DVDD VREF set to 3.3 V for 2.5 A full-scale current regulation Step pulse driven by PWM Direction and current limit set by SPI registers"
- note removed: "BED WING SPAN MOTOR DRIVER"
- note removed: "Designed for 12 V DC stepper motor load up to 1.8 A rms (2.5 A peak)"
- note removed: "Device controlled over SPI so STEP and DIR not used VREF tied to DVDD for full-scale current limit, can be scaled down with TRQ_DAC register"
- moved on the sheet: C35, C36, C37, C38, C39, C40, J11, U7

Commit message: Further refinement.
Parts:
- renumbered C33 to C38, C34 to C39, C35 to C40, C36 to C41, C37 to C42, C38 to C43, C39 to C44, C40 to C45, J11 to J12
