File: hardware/v1/bed-lift.kicad_pcb (KiCad board)
At the start: 4 copper layers, 195 x 45 mm, 154 parts, among them J1 SM04B-SRSS-TB, J10 Molex Mini Fit Jr 39-30-1060, J11 Molex Mini Fit Jr 39-30-1060, J12 S4B-XH-A, J13 S4B-XH-A, J14 S4B-XH-A, J15 S4B-XH-A, J2 S2P-VH, J3 SM04B-SRSS-TB, J4 S3B-XH-A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

Commit message: Finalize for production of v1.0 revision.
Parts:
- D2, D3, D6, D7: value PESD5V0S2UAT -> PESD5V0L2UU; footprint Package_TO_SOT_SMD:SOT-23 -> Package_TO_SOT_SMD:SOT-323_SC-70
- moved D2 0.25 mm to (65.8, 85.2)
- moved D3 0.25 mm to (46.0, 85.2)
- moved D6 0.25 mm to (108.5, 76.5)
- moved D7 0.25 mm to (132.5, 76.5)
Routing:
- net GND: track 158.4 -> 156.9 mm
- net Net-(J4-Pin_2): track 7.75 -> 6.74 mm
- net Net-(J7-Pin_2): track 6.98 -> 7.56 mm
Other:
- board text added: "1: GND 2: SPN1_LA 3: SPN1_LB 4: SPN2_LA 5: SPN2_LB 6: 5V"
- board text added: "1:HALL2 2:GND 3:5V 4:OUT2 5:OUT1 6:HALL1"
- board text added: "BT0 (NC) PA12 PB12 SCL2 3V3 5V 12V"
- board text added: "RST PA15 PA11 PB13 SDA2 GND GND GND"
- board text removed: "1: GND 2: SPN1_LA 3: SPN1_LB 4: SPN2_LA 5: SPN2_LB 6: VHALL"
- board text removed: "1:HALL2 2:GND 3:VHALL 4:OUT2 5:OUT1 6:HALL1"
- board text removed: "BT0 (NC) PA12 PB12 SCL 3V3 5V 12V"
- board text removed: "RST PA15 PA11 PB13 SDA GND GND GND"
