File: hardware/v1/lift.kicad_sch (KiCad schematic)
At the start: 16 parts, among them J10 Molex Mini Fit Jr 39-30-1060, U5 DRV8874PWPR

Commit message: Finalize for production of v1.0 revision.
Parts:
- C18: MPN 4700250508R00 -> (none); Part (none) -> 4700250508R00
- D6: value PESD5V0S2UAT -> PESD5V0L2UU; footprint Package_TO_SOT_SMD:SOT-23 -> Package_TO_SOT_SMD:SOT-323_SC-70; FT Rotation Offset (none) -> 180; LCSC C552572 -> C78769; LCSC Alternative (none) -> C28646364
Changed lines of the file:
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@@
 			)
 		)
-		(property "MPN" "4700250508R00"
-			(at 108.331 54.7596 0)
-			(effects
-				(font
-					(size 1.27 1.27)
-				)
-				(justify left)
+		(property "Part" "4700250508R00"
+			(at 105.41 50.8 0)
+			(effects
+				(font
+					(size 1.27 1.27)
+				)
 				(hide yes)
 			)
@@
 			)
 		)
-		(property "Value" "PESD5V0S2UAT"
+		(property "Value" "PESD5V0L2UU"
 			(at 186.182 134.4986 90)
 			(effects
@@
 			)
 		)
-		(property "Footprint" "Package_TO_SOT_SMD:SOT-23"
+		(property "Footprint" "Package_TO_SOT_SMD:SOT-323_SC-70"
 			(at 181.61 134.62 0)
 			(effects
@@
 			)
 		)
-		(property "Datasheet" "https://assets.nexperia.com/documents/data-sheet/PESD5V0S2UAT.pdf"
+		(property "Datasheet" "https://assets.nexperia.com/documents/data-sheet/PESD5V0L2UU.pdf"
 			(at 181.61 134.62 0)
 			(effects
@@
 			)
 		)
-		(property "LCSC" "C552572"
+		(property "LCSC" "C78769"
 			(at 181.61 133.35 0)
 			(effects
 				(font
+					(size 1.27 1.27)
+				)
+				(hide yes)
+			)
+		)
+		(property "LCSC Alternative" "C28646364"
+			(at 181.61 133.35 90)
+			(effects
+				(font
+					(size 1.27 1.27)
+				)
+				(hide yes)
+			)
+		)
+		(property "FT Rotation Offset" "180"
+			(at 181.61 133.35 90)
+			(effects
+				(font
