File: hardware/v1/span.kicad_sch (KiCad schematic)
At the start: 10 parts, among them J12 S4B-XH-A, U7 DRV8434SPWPR

Commit message: Finalize for production of v1.0 revision.
Parts:
- C38: MPN 4700250508R00 -> (none); Part (none) -> 4700250508R00
Changed lines of the file:
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@@
 			)
 		)
-		(property "MPN" "4700250508R00"
-			(at 89.281 73.8096 0)
+		(property "Part" "4700250508R00"
+			(at 86.36 69.85 0)
 			(effects
 				(font
 					(size 1.27 1.27)
 				)
-				(justify left)
 				(hide yes)
 			)
